File: mfk60_middle_plate.kicad_pcb (KiCad board)
At the start: 2 copper layers, 300 x 95.2 mm, 78 parts, among them SW1 COL1_ROW1, SW10 COL10_ROW1, SW11 COL11_ROW1, SW12 COL12_ROW1, SW13 COL13_ROW1, SW14 COL14_ROW1, SW15 COL1_ROW2, SW16 COL2_ROW2, SW17 COL3_ROW2, SW18 COL4_ROW2, SW19 COL5_ROW2, SW2 COL2_ROW1, SW20 COL6_ROW2, SW21 COL7_ROW2, SW22 COL8_ROW2, SW23 COL9_ROW2, SW24 COL10_ROW2, SW25 COL11_ROW2, SW26 COL12_ROW2, SW27 COL13_ROW2, SW28 COL14_ROW2, SW29 COL1_ROW3, SW3 COL3_ROW1, SW30 COL2_ROW3, SW31 COL3_ROW3, SW32 COL4_ROW3, SW33 COL5_ROW3, SW34 COL6_ROW3, SW35 COL7_ROW3, SW36 COL8_ROW3, SW37 COL9_ROW3, SW38 COL10_ROW3, SW39 COL11_ROW3, SW4 COL4_ROW1, SW40 COL12_ROW3, SW41 COL13_ROW3, SW42 COL1_ROW4, SW43 COL2_ROW4, SW44 COL3_ROW4, SW45 COL4_ROW4, SW46 COL5_ROW4, SW47 COL6_ROW4, SW48 COL7_ROW4, SW49 COL8_ROW4, SW5 COL5_ROW1, SW50 COL9_ROW4, SW51 COL10_ROW4, SW52 COL11_ROW4, SW53 COL12_ROW4, SW54 COL13_ROW4, SW55 COL1_ROW5, SW56 COL2_ROW5, SW57 COL3_ROW5, SW58 COL7_ROW5, SW59 COL8_ROW5, SW6 COL6_ROW1, SW60 COL9_ROW5, SW61 COL10_ROW5, SW7 COL7_ROW1, SW8 COL8_ROW1, SW9 COL9_ROW1, T1 Tab, T2 Tab, T3 Tab, T4 Tab, T5 Tab, T6 Tab, T7 Tab

Commit message: Adjust JLC text position and add it to script.
Other:
- board text added: "JLCJLCJLCJLC"
Changed lines of the file:
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@@
   (gr_arc (start 137.3 25) (mid 138.714214 25.585786) (end 139.3 27)
     (stroke (width 0.1) (type default)) (layer "Edge.Cuts"))
+  (gr_text "JLCJLCJLCJLC" (at 297.653125 110.725) (layer "F.SilkS")
+    (effects (font (size 1 1) (thickness 0.15)) (justify bottom))
+  )
 )
