File: mfk60_middle_plate.kicad_pcb (KiCad board)
At the start: 2 copper layers, 300 x 95.2 mm, 78 parts, among them SW1 COL1_ROW1, SW10 COL10_ROW1, SW11 COL11_ROW1, SW12 COL12_ROW1, SW13 COL13_ROW1, SW14 COL14_ROW1, SW15 COL1_ROW2, SW16 COL2_ROW2, SW17 COL3_ROW2, SW18 COL4_ROW2, SW19 COL5_ROW2, SW2 COL2_ROW1, SW20 COL6_ROW2, SW21 COL7_ROW2, SW22 COL8_ROW2, SW23 COL9_ROW2, SW24 COL10_ROW2, SW25 COL11_ROW2, SW26 COL12_ROW2, SW27 COL13_ROW2, SW28 COL14_ROW2, SW29 COL1_ROW3, SW3 COL3_ROW1, SW30 COL2_ROW3, SW31 COL3_ROW3, SW32 COL4_ROW3, SW33 COL5_ROW3, SW34 COL6_ROW3, SW35 COL7_ROW3, SW36 COL8_ROW3, SW37 COL9_ROW3, SW38 COL10_ROW3, SW39 COL11_ROW3, SW4 COL4_ROW1, SW40 COL12_ROW3, SW41 COL13_ROW3, SW42 COL1_ROW4, SW43 COL2_ROW4, SW44 COL3_ROW4, SW45 COL4_ROW4, SW46 COL5_ROW4, SW47 COL6_ROW4, SW48 COL7_ROW4, SW49 COL8_ROW4, SW5 COL5_ROW1, SW50 COL9_ROW4, SW51 COL10_ROW4, SW52 COL11_ROW4, SW53 COL12_ROW4, SW54 COL13_ROW4, SW55 COL1_ROW5, SW56 COL2_ROW5, SW57 COL3_ROW5, SW58 COL7_ROW5, SW59 COL8_ROW5, SW6 COL6_ROW1, SW60 COL9_ROW5, SW61 COL10_ROW5, SW7 COL7_ROW1, SW8 COL8_ROW1, SW9 COL9_ROW1, T1 Tab, T2 Tab, T3 Tab, T4 Tab, T5 Tab, T6 Tab, T7 Tab

Commit message: Add missing npth for USB-C socket.
Parts:
- added J1: USB_C_Receptacle_USB2.0, Connector_Additions:USB_C_Receptacle_HRO_TYPE-C-31-M-12_Middle_Plate, B.Cu at (44.0, 28.6)
- added J4: USB_C_Receptacle_USB2.0, Connector_Additions:USB_C_Receptacle_HRO_TYPE-C-31-M-12_Middle_Plate, B.Cu at (291.7, 28.6)
Changed lines of the file:
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@@
       (stroke (width 0.15) (type default)) (layer "Edge.Cuts"))
+  )
+  (footprint "Connector_Additions:USB_C_Receptacle_HRO_TYPE-C-31-M-12_Middle_Plate" (layer "B.Cu")
+    (at 291.7 28.65)
+    (descr "USB Type-C receptacle for USB 2.0 and PD, http://www.krhro.com/uploads/soft/180320/1-1P320120243.pdf")
+    (tags "usb usb-c 2.0 pd")
+    (property "LCSC" "C2982555")
+    (property "Matrix" "")
+    (property "Sheetfile" "mfk60_right.kicad_sch")
+    (property "Sheetname" "Righ")
+    (property "ki_description" "USB 2.0-only 16P Type-C Receptacle connector")
+    (property "ki_keywords" "usb universal serial bus type-C USB2.0")
+    (attr smd board_only)
+    (fp_text reference "J4" (at 0 5.645 180) (layer "B.SilkS") hide
+        (effects (font (size 1 1) (thickness 0.15)) (justify mirror))
+    )
+    (fp_text value "USB_C_Receptacle_USB2.0" (at 0 -5.1 180) (layer "B.Fab")
+        (effects (font (size 1 1) (thickness 0.15)) (justify mirror))
+    )
+    (fp_text user "${REFERENCE}" (at 0 0 180) (layer "B.Fab")
+        (effects (font (size 1 1) (thickness 0.15)) (justify mirror))
+    )
+    (fp_line (start -5.32 -4.15) (end 5.32 -4.15)
+      (stroke (width 0.05) (type solid)) (layer "B.CrtYd"))
+    (fp_line (start -5.32 5.27) (end -5.32 -4.15)
+      (stroke (width 0.05) (type solid)) (layer "B.CrtYd"))
+    (fp_line (start -5.32 5.27) (end 5.32 5.27)
+      (stroke (width 0.05) (type solid)) (layer "B.CrtYd"))
+    (fp_line (start 5.32 5.27) (end 5.32 -4.15)
+      (stroke (width 0.05) (type solid)) (layer "B.CrtYd"))
+    (fp_line (start -4.47 -3.65) (end 4.47 -3.65)
+      (stroke (width 0.1) (type solid)) (layer "B.Fab"))
+    (fp_line (start -4.47 3.65) (end -4.47 -3.65)
+      (stroke (width 0.1) (type solid)) (layer "B.Fab"))
+    (fp_line (start -4.47 3.65) (end 4.47 3.65)
+      (stroke (width 0.1) (type solid)) (layer "B.Fab"))
+    (fp_line (start 4.47 3.65) (end 4.47 -3.65)
+      (stroke (width 0.1) (type solid)) (layer "B.Fab"))
+    (pad "" np_thru_hole oval (at -4.32 -1.05) (size 1.4 2) (drill oval 1.4 2) (layers "F&B.Cu" "*.Mask"))
+    (pad "" np_thru_hole oval (at -4.32 3.13) (size 1.4 2.5) (drill oval 1.4 2.5) (layers "F&B.Cu" "*.Mask"))
+    (pad "" np_thru_hole oval (at 4.32 -1.05) (size 1.4 2) (drill oval 1.4 2) (layers "F&B.Cu" "*.Mask"))
+    (pad "" np_thru_hole oval (at 4.32 3.13) (size 1.4 2.5) (drill oval 1.4 2.5) (layers "F&B.Cu" "*.Mask"))
+    (model "${KICAD6_3DMODEL_DIR}/Connector_USB.3dshapes/USB_C_Receptacle_HRO_TYPE-C-31-M-12.wrl"
+      (offset (xyz 0 0 0))
+      (scale (xyz 1 1 1))
+      (rotate (xyz 0 0 0))
+    )
   )
   (footprint "MountingHole:MountingHole_2.2mm_M2" (layer "B.Cu")
@@
     (pad "" np_thru_hole circle (at 0 0 180) (size 2.2 2.2) (drill 2.2) (layers "*.Cu" "*.Mask"))
   )
+  (footprint "Connector_Additions:USB_C_Receptacle_HRO_TYPE-C-31-M-12_Middle_Plate" (layer "B.Cu")
+    (at 44.05 28.65)
+    (descr "USB Type-C receptacle for USB 2.0 and PD, http://www.krhro.com/uploads/soft/180320/1-1P320120243.pdf")
+    (tags "usb usb-c 2.0 pd")
+    (property "LCSC" "C2982555")
+    (property "Matrix" "")
+    (property "Sheetfile" "mfk60_left.kicad_sch")
+    (property "Sheetname" "Left")
+    (property "ki_description" "USB 2.0-only 16P Type-C Receptacle connector")
+    (property "ki_keywords" "usb universal serial bus type-C USB2.0")
+    (attr smd board_only)
+    (fp_text reference "J1" (at 0 5.645 180) (layer "B.SilkS") hide
+        (effects (font (size 1 1) (thickness 0.15)) (justify mirror))
+    )
+    (fp_text value "USB_C_Receptacle_USB2.0" (at 0 -5.1 180) (layer "B.Fab")
+        (effects (font (size 1 1) (thickness 0.15)) (justify mirror))
+    )
+    (fp_text user "${REFERENCE}" (at 0 0 180) (layer "B.Fab")
+        (effects (font (size 1 1) (thickness 0.15)) (justify mirror))
+    )
+    (fp_line (start -5.32 -4.15) (end 5.32 -4.15)
+      (stroke (width 0.05) (type solid)) (layer "B.CrtYd"))
+    (fp_line (start -5.32 5.27) (end -5.32 -4.15)
+      (stroke (width 0.05) (type solid)) (layer "B.CrtYd"))
+    (fp_line (start -5.32 5.27) (end 5.32 5.27)
+      (stroke (width 0.05) (type solid)) (layer "B.CrtYd"))
+    (fp_line (start 5.32 5.27) (end 5.32 -4.15)
+      (stroke (width 0.05) (type solid)) (layer "B.CrtYd"))
+    (fp_line (start -4.47 -3.65) (end 4.47 -3.65)
+      (stroke (width 0.1) (type solid)) (layer "B.Fab"))
+    (fp_line (start -4.47 3.65) (end -4.47 -3.65)
+      (stroke (width 0.1) (type solid)) (layer "B.Fab"))
+    (fp_line (start -4.47 3.65) (end 4.47 3.65)
+      (stroke (width 0.1) (type solid)) (layer "B.Fab"))
+    (fp_line (start 4.47 3.65) (end 4.47 -3.65)
+      (stroke (width 0.1) (type solid)) (layer "B.Fab"))
+    (pad "" np_thru_hole oval (at -4.32 -1.05) (size 1.4 2) (drill oval 1.4 2) (layers "F&B.Cu" "*.Mask"))
+    (pad "" np_thru_hole oval (at -4.32 3.13) (size 1.4 2.5) (drill oval 1.4 2.5) (layers "F&B.Cu" "*.Mask"))
+    (pad "" np_thru_hole oval (at 4.32 -1.05) (size 1.4 2) (drill oval 1.4 2) (layers "F&B.Cu" "*.Mask"))
+    (pad "" np_thru_hole oval (at 4.32 3.13) (size 1.4 2.5) (drill oval 1.4 2.5) (layers "F&B.Cu" "*.Mask"))
+    (model "${KICAD6_3DMODEL_DIR}/Connector_USB.3dshapes/USB_C_Receptacle_HRO_TYPE-C-31-M-12.wrl"
+      (offset (xyz 0 0 0))
+      (scale (xyz 1 1 1))
+      (rotate (xyz 0 0 0))
+    )
+  )
   (footprint "MountingHole:MountingHole_2.2mm_M2" (layer "B.Cu")
