File: mfk60_right.kicad_sch (KiCad schematic)
At the start: 31 parts, among them J1 USB_C_Receptacle_USB2.0, J2 ISP, J3 TRRS Jack, SW1 RST, T4 Tab, T5 Tab, T6 Tab, T7 Tab, U1 ATmega32U4-M, Y1 16M

Commit message: Add pull-up resistor on left side.
Parts:
- renumbered R13 to R12
Connections:
- net SPLIT_HAND renamed R_SPLIT_HAND
Changed lines of the file:
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@@
     )
   )
-  (global_label "SPLIT_HAND" (shape input) (at 248.92 96.52 0) (fields_autoplaced)
-    (effects (font (size 1.27 1.27)) (justify left))
-    (property "Intersheetrefs" "${INTERSHEET_REFS}" (at 262.9724 96.52 0)
+  (global_label "R_SPLIT_HAND" (shape input) (at 248.92 96.52 0) (fields_autoplaced)
+    (effects (font (size 1.27 1.27)) (justify left))
+    (property "Intersheetrefs" "${INTERSHEET_REFS}" (at 265.21 96.52 0)
       (effects (font (size 1.27 1.27)) (justify left) hide)
     )
@@
     )
   )
-  (global_label "SPLIT_HAND" (shape input) (at 143.51 128.27 0) (fields_autoplaced)
-    (effects (font (size 1.27 1.27)) (justify left))
-    (property "Intersheetrefs" "${INTERSHEET_REFS}" (at 157.5624 128.27 0)
+  (global_label "R_SPLIT_HAND" (shape input) (at 143.51 128.27 0) (fields_autoplaced)
+    (effects (font (size 1.27 1.27)) (justify left))
+    (property "Intersheetrefs" "${INTERSHEET_REFS}" (at 159.8 128.27 0)
       (effects (font (size 1.27 1.27)) (justify left) hide)
     )
@@
   (symbol (lib_id "Device:R_Small") (at 138.43 135.89 180) (unit 1)
     (in_bom yes) (on_board yes) (dnp no) (fields_autoplaced)
-    (property "Reference" "R13" (at 140.97 134.62 0)
+    (property "Reference" "R12" (at 140.97 134.62 0)
       (effects (font (size 1.27 1.27)) (justify right))
     )
@@
       (project "mfk60"
         (path "/5884af6c-f4a4-4f6a-8d5a-73da30f3acf7/9b5d010c-c128-4221-9df0-679e0e88f90c"
-          (reference "R13") (unit 1)
+          (reference "R12") (unit 1)
         )
       )
@@
       (project "mfk60"
         (path "/5884af6c-f4a4-4f6a-8d5a-73da30f3acf7/9b5d010c-c128-4221-9df0-679e0e88f90c"
-          (reference "R7") (unit 1)
+          (reference "R13") (unit 1)
         )
       )
@@
       (project "mfk60"
         (path "/5884af6c-f4a4-4f6a-8d5a-73da30f3acf7/9b5d010c-c128-4221-9df0-679e0e88f90c"
-          (reference "R12") (unit 1)
-        )
-      )
+          (reference "R14") (unit 1)
+        )
+      )

Commit message: FIX: key and diode value
Parts:
- J3: LCSC (none) -> C431535
- SW1: LCSC (none) -> C139797
Changed lines of the file:
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@@
+      (effects (font (size 1.27 1.27)) hide)
+    )
+    (property "Matrix" "" (at 101.6 156.21 0)
       (effects (font (size 1.27 1.27)) hide)
     )
@@
     )
     (property "LCSC" "" (at 38.1 166.37 0)
+      (effects (font (size 1.27 1.27)) hide)
+    )
+    (property "Matrix" "" (at 38.1 166.37 0)
       (effects (font (size 1.27 1.27)) hide)
     )
@@
       (effects (font (size 1.27 1.27)) hide)
     )
+    (property "Matrix" "" (at 69.85 35.56 0)
+      (effects (font (size 1.27 1.27)) hide)
+    )
     (pin "1")
     (pin "2")
@@
       (effects (font (size 1.27 1.27)) hide)
     )
+    (property "Matrix" "" (at 119.38 69.85 0)
+      (effects (font (size 1.27 1.27)) hide)
+    )
     (pin "1")
     (pin "2")
@@
       (effects (font (size 1.27 1.27)) hide)
     )
+    (property "Matrix" "" (at 125.73 184.15 0)
+      (effects (font (size 1.27 1.27)) hide)
+    )
     (instances
       (project "mfk60"
@@
       (effects (font (size 1.27 1.27)) hide)
     )
+    (property "Matrix" "" (at 60.96 109.22 0)
+      (effects (font (size 1.27 1.27)) hide)
+    )
     (pin "1")
     (pin "2")
@@
       (effects (font (size 1.27 1.27)) hide)
     )
+    (property "Matrix" "" (at 60.96 96.52 0)
+      (effects (font (size 1.27 1.27)) hide)
+    )
     (pin "1")
     (pin "2")
@@
       (effects (font (size 1.27 1.27)) hide)
     )
+    (property "Matrix" "" (at 101.6 168.91 0)
+      (effects (font (size 1.27 1.27)) hide)
+    )
     (instances
       (project "mfk60"
@@
     )
     (property "Datasheet" "~" (at 125.73 168.91 0)
+      (effects (font (size 1.27 1.27)) hide)
+    )
+    (property "Matrix" "" (at 125.73 168.91 0)
       (effects (font (size 1.27 1.27)) hide)
     )
@@
       (effects (font (size 1.27 1.27)) hide)
     )
+    (property "Matrix" "" (at 125.73 176.53 0)
+      (effects (font (size 1.27 1.27)) hide)
+    )
     (instances
       (project "mfk60"
@@
     )
     (property "Datasheet" "~" (at 125.73 156.21 0)
+      (effects (font (size 1.27 1.27)) hide)
+    )
+    (property "Matrix" "" (at 125.73 156.21 0)
       (effects (font (size 1.27 1.27)) hide)
     )
@@
     )
     (property "LCSC" "C17414" (at 138.43 135.89 0)
+      (effects (font (size 1.27 1.27)) hide)
+    )
+    (property "Matrix" "" (at 138.43 135.89 0)
       (effects (font (size 1.27 1.27)) hide)
     )
@@
       (effects (font (size 1.27 1.27)) hide)
     )
+    (property "Matrix" "" (at 101.6 184.15 0)
+      (effects (font (size 1.27 1.27)) hide)
+    )
     (instances
       (project "mfk60"
@@
       (effects (font (size 1.27 1.27)) hide)
     )
+    (property "Matrix" "" (at 101.6 176.53 0)
+      (effects (font (size 1.27 1.27)) hide)
+    )
     (instances
       (project "mfk60"
@@
     )
     (property "Datasheet" "~" (at 101.6 162.56 0)
+      (effects (font (size 1.27 1.27)) hide)
+    )
+    (property "Matrix" "" (at 101.6 162.56 0)
       (effects (font (size 1.27 1.27)) hide)
     )
@@
       (effects (font (size 1.27 1.27)) hide)
     )
+    (property "Matrix" "" (at 62.23 88.9 0)
+      (effects (font (size 1.27 1.27)) hide)
+    )
     (pin "1")
     (pin "2")
@@
       (effects (font (size 1.27 1.27)) hide)
     )
+    (property "Matrix" "" (at 119.38 62.23 0)
+      (effects (font (size 1.27 1.27)) hide)
+    )
     (pin "1")
     (pin "2")
@@
       (effects (font (size 1.27 1.27)) hide)
     )
+    (property "Matrix" "" (at 100.33 35.56 0)
+      (effects (font (size 1.27 1.27)) hide)
+    )
     (pin "1")
     (pin "2")
@@
     )
     (property "LCSC" "C49678" (at 90.17 35.56 0)
+      (effects (font (size 1.27 1.27)) hide)
+    )
+    (property "Matrix" "" (at 90.17 35.56 0)
       (effects (font (size 1.27 1.27)) hide)
     )
@@
     )
     (property "LCSC" "C112161" (at 226.06 91.44 0)
+      (effects (font (size 1.27 1.27)) hide)
+    )
+    (property "Matrix" "" (at 226.06 91.44 0)
       (effects (font (size 1.27 1.27)) hide)
     )
@@
       (effects (font (size 1.27 1.27)) hide)
     )
+    (property "Matrix" "" (at 125.73 162.56 0)
+      (effects (font (size 1.27 1.27)) hide)
+    )
     (instances
       (project "mfk60"
@@
       (effects (font (size 1.27 1.27)) hide)
     )
+    (property "Matrix" "" (at 132.08 66.04 0)
+      (effects (font (size 1.27 1.27)) hide)
+    )
     (pin "1")
     (pin "2")
@@
     )
     (property "LCSC" "C17561" (at 60.96 104.14 0)
+      (effects (font (size 1.27 1.27)) hide)
+    )
+    (property "Matrix" "" (at 60.96 104.14 0)
       (effects (font (size 1.27 1.27)) hide)
     )
@@
       (effects (font (size 1.27 1.27)) hide)
     )
+    (property "Matrix" "" (at 203.2 46.99 0)
+      (effects (font (size 1.27 1.27)) hide)
+    )
     (pin "1")
     (pin "2")
@@
       (effects (font (size 1.27 1.27)) hide)
     )
+    (property "Matrix" "" (at 245.11 138.43 0)
+      (effects (font (size 1.27 1.27)) hide)
+    )
     (pin "1")
     (pin "2")
@@
     )
     (property "LCSC" "C2982555" (at 31.75 104.14 0)
+      (effects (font (size 1.27 1.27)) hide)
+    )
+    (property "Matrix" "" (at 31.75 104.14 0)
       (effects (font (size 1.27 1.27)) hide)
     )
@@
       (effects (font (size 1.524 1.524)) hide)
     )
-    (property "LCSC" "" (at 121.92 105.41 0)
+    (property "LCSC" "C431535" (at 121.92 105.41 0)
+      (effects (font (size 1.27 1.27)) hide)
+    )
+    (property "Matrix" "" (at 121.92 105.41 0)
       (effects (font (size 1.27 1.27)) hide)
     )
@@
       (effects (font (size 1.27 1.27)) hide)
     )
+    (property "Matrix" "" (at 60.96 93.98 0)
+      (effects (font (size 1.27 1.27)) hide)
+    )
     (pin "1")
     (pin "2")
@@
       (effects (font (size 1.27 1.27)) hide)
     )
+    (property "Matrix" "" (at 203.2 91.44 0)
+      (effects (font (size 1.27 1.27)) hide)
+    )
     (pin "1")
     (pin "2")
@@
       (effects (font (size 1.27 1.27)) hide)
     )
+    (property "Matrix" "" (at 80.01 35.56 0)
+      (effects (font (size 1.27 1.27)) hide)
+    )
     (pin "1")
     (pin "2")
@@
       (effects (font (size 1.27 1.27)) hide)
     )
+    (property "Matrix" "" (at 142.24 33.02 0)
+      (effects (font (size 1.27 1.27)) hide)
+    )
+    (property "LCSC" "C139797" (at 142.24 33.02 0)
+      (effects (font (size 1.27 1.27)) hide)
+    )
